File: code/transmitter.kicad_sch (KiCad schematic)
At the start: 16 parts, among them IC1 BD9E303UEFJ-LBE2, J1 Conn_01x02, J2 Conn_01x01, J3 Conn_01x01, J4 Conn_01x01, J5 Conn_01x02, U2 NC7SVU04P5X, U4 DRV8220DRLR

Commit message: new buck boi
Parts:
- removed IC1: BD9E303UEFJ-LBE2, SOIC127P600X100-9N, symbol New_Library:BD9E303UEFJ-LBE2
- added C_IN_buck, C_OUT_buck, C_SS, C_boot: C, symbol Device:C
- added D5: SB120, Diode_THT:D_DO-41_SOD81_P10.16mm_Horizontal, symbol Diode:SB120
- added L1: L, symbol Device:L
- added R_FBB, R_FBT, R_T_buck: R, symbol Device:R
- added U1: LMR14050SDDAR, DDA0008E_N, symbol New_Library:LMR14050SDDAR
Connections:
- net 0: now also C_IN_buck.2, C_OUT_buck.2, C_SS.2, D5.2 (A), R_FBB.2, R_T_buck.1, U1.7 (GND), U1.9 (PAD)
- net at C1.1, C3.1, D3.1 (K)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: now also C_IN_buck.1, U1.2 (VIN), U1.3 (EN)
- net at C2.1, U4.5 (VM): now also C_OUT_buck.1, L1.2, R_FBT.1
- new net: C_boot.1, U1.1 (BOOT)
- new net: R_T_buck.2, U1.4 (RT_SYNC)
- new net: R_FBB.1, R_FBT.2, U1.5 (FB)
- new net: C_SS.1, U1.6 (SS)
- new net: C_boot.2, D5.1 (K), L1.1, U1.8 (SW)
Other:
- moved on the sheet: C3
